Commit message: Fix problem where either the world or the robot can be spawned in gazebo

File: ros2_ws/src/milo_sim/urdf/milo_core.urdf.xacro (robot description, xacro)
@@ -1,18 +1,18 @@
 <?xml version="1.0"?>
-<robot xmlns:xacro="http://www.ros.org/wiki/xacro" >
+<robot xmlns:xacro="http://www.ros.org/wiki/xacro">
   <!-- Include useful macros -->
-  <xacro:include filename="inertial_macros.xacro"/>
-  <xacro:include filename="colors.xacro"/>
+  <xacro:include filename="inertial_macros.xacro" />
+  <xacro:include filename="colors.xacro" />
   <!-- Define the robot's properties -->
-  <xacro:property name="chassis_length" value="0.26"/>
-  <xacro:property name="chassis_width" value="0.26"/>
-  <xacro:property name="chassis_height" value="0.05"/>
-  <xacro:property name="chassis_mass" value="0.350"/>
-  <xacro:property name="wheel_axis_offset_x" value="0.04"/>
-  <xacro:property name="wheel_axis_offset_z" value="0.01"/>
-  <xacro:property name="wheel_radius" value="0.03"/>
-  <xacro:property name="wheel_thickness" value="0.025"/>
-  <xacro:property name="ldr_inter_offset" value="0.02"/>
-  <xacro:property name="ldr_height" value="0.01"/>
+  <xacro:property name="chassis_length" value="0.26" />
+  <xacro:property name="chassis_width" value="0.26" />
+  <xacro:property name="chassis_height" value="0.05" />
+  <xacro:property name="chassis_mass" value="0.350" />
+  <xacro:property name="wheel_axis_offset_x" value="0.04" />
+  <xacro:property name="wheel_axis_offset_z" value="0.01" />
+  <xacro:property name="wheel_radius" value="0.03" />
+  <xacro:property name="wheel_thickness" value="0.025" />
+  <xacro:property name="ldr_inter_offset" value="0.02" />
+  <xacro:property name="ldr_height" value="0.01" />
   <!-- World link without inertia required by rviz -->
   <link name="base_link">
@@ -20,248 +20,253 @@
   <!-- CHASSIS -->
   <joint name="chassis_joint" type="fixed">
-    <parent link="base_link"/>
-    <child link="chassis_link"/>
-    <origin xyz="${-chassis_length/2} 0.0 0.0" rpy="0.0 0.0 0.0"/>
+    <parent link="base_link" />
+    <child link="chassis_link" />
+    <origin xyz="${-chassis_length/2} 0.0 0.1" rpy="0.0 0.0 0.0" />
   </joint>
   <link name="chassis_link">
     <visual>
       <geometry>
-        <box size="${chassis_length} ${chassis_width} ${chassis_height}"/>
-      </geometry>
-      <origin xyz="${chassis_length/2} 0 ${chassis_height/2}"/>
+        <box size="${chassis_length} ${chassis_width} ${chassis_height}" />
+      </geometry>
+      <origin xyz="${chassis_length/2} 0 ${chassis_height/2}" />
       <material name="white" />
     </visual>
     <collision>
       <geometry>
-        <box size="${chassis_length} ${chassis_width} ${chassis_height}"/>
-      </geometry>
-      <origin xyz="${chassis_length/2} 0 ${chassis_height/2}"/>
-    </collision>
-    <xacro:inertial_box mass="${chassis_mass}" x="${chassis_length}" y="${chassis_width}" z="${chassis_height}">
-      <origin xyz="${chassis_length/2} 0 ${chassis_height/2}"/>
+        <box size="${chassis_length} ${chassis_width} ${chassis_height}" />
+      </geometry>
+      <origin xyz="${chassis_length/2} 0 ${chassis_height/2}" />
+    </collision>
+    <xacro:inertial_box mass="${chassis_mass}" x="${chassis_length}" y="${chassis_width}"
+      z="${chassis_height}">
+      <origin xyz="${chassis_length/2} 0 ${chassis_height/2}" />
     </xacro:inertial_box>
   </link>
   <!-- WHEELS (looked at from the front of the robot) -->
   <joint name="BR_wheel_joint" type="continuous">
-    <parent link="chassis_link"/>
-    <child link="BR_wheel_link"/>
-    <origin xyz="${wheel_axis_offset_x} ${chassis_width/2} ${wheel_axis_offset_z}" rpy="${pi/2} 0 0"/>
-    <axis xyz="0.0 0.0 1"/>
+    <parent link="chassis_link" />
+    <child link="BR_wheel_link" />
+    <origin xyz="${wheel_axis_offset_x} ${chassis_width/2} ${wheel_axis_offset_z}" rpy="${pi/2} 0 0" />
+    <axis xyz="0.0 0.0 1" />
   </joint>
   <link name="BR_wheel_link">
     <visual>
       <geometry>
-        <cylinder radius="${wheel_radius}" length="${wheel_thickness}"/>
-      </geometry>
-      <origin xyz="0 0 ${-wheel_thickness/2}"/>
-      <material name="black" />
-    </visual>
-    <collision>
-      <geometry>
-        <cylinder radius="${wheel_radius}" length="${wheel_thickness}"/>
-      </geometry>
-      <origin xyz="0 0 ${-wheel_thickness/2}"/>
+        <cylinder radius="${wheel_radius}" length="${wheel_thickness}" />
+      </geometry>
+      <origin xyz="0 0 ${-wheel_thickness/2}" />
+      <material name="black" />
+    </visual>
+    <collision>
+      <geometry>
+        <cylinder radius="${wheel_radius}" length="${wheel_thickness}" />
+      </geometry>
+      <origin xyz="0 0 ${-wheel_thickness/2}" />
     </collision>
     <xacro:inertial_cylinder mass="0.020" radius="${wheel_radius}" length="${wheel_thickness}">
-      <origin xyz="0 0 ${-wheel_thickness/2}"/>
+      <origin xyz="0 0 ${-wheel_thickness/2}" />
     </xacro:inertial_cylinder>
   </link>
   <joint name="BL_wheel_joint" type="continuous">
-    <parent link="chassis_link"/>
-    <child link="BL_wheel_link"/>
-    <origin xyz="${wheel_axis_offset_x} ${-chassis_width/2} ${wheel_axis_offset_z}" rpy="${pi/2} 0 0"/>
-    <axis xyz="0.0 0.0 1"/>
+    <parent link="chassis_link" />
+    <child link="BL_wheel_link" />
+    <origin xyz="${wheel_axis_offset_x} ${-chassis_width/2} ${wheel_axis_offset_z}"
+      rpy="${pi/2} 0 0" />
+    <axis xyz="0.0 0.0 1" />
   </joint>
   <link name="BL_wheel_link">
     <visual>
       <geometry>
-        <cylinder radius="${wheel_radius}" length="${wheel_thickness}"/>
-      </geometry>
-      <origin xyz="0 0 ${wheel_thickness/2}"/>
-      <material name="black" />
-    </visual>
-    <collision>
-      <geometry>
-        <cylinder radius="${wheel_radius}" length="${wheel_thickness}"/>
-      </geometry>
-      <origin xyz="0 0 ${wheel_thickness/2}"/>
+        <cylinder radius="${wheel_radius}" length="${wheel_thickness}" />
+      </geometry>
+      <origin xyz="0 0 ${wheel_thickness/2}" />
+      <material name="black" />
+    </visual>
+    <collision>
+      <geometry>
+        <cylinder radius="${wheel_radius}" length="${wheel_thickness}" />
+      </geometry>
+      <origin xyz="0 0 ${wheel_thickness/2}" />
     </collision>
     <xacro:inertial_cylinder mass="0.020" radius="${wheel_radius}" length="${wheel_thickness}">
-      <origin xyz="0 0 ${wheel_thickness/2}"/>
+      <origin xyz="0 0 ${wheel_thickness/2}" />
     </xacro:inertial_cylinder>
   </link>
   <joint name="FL_wheel_joint" type="continuous">
-    <parent link="chassis_link"/>
-    <child link="FL_wheel_link"/>
-    <origin xyz="${chassis_length - wheel_axis_offset_x} ${-chassis_width/2} ${wheel_axis_offset_z}" rpy="${pi/2} 0 0"/>
-    <axis xyz="0.0 0.0 1"/>
+    <parent link="chassis_link" />
+    <child link="FL_wheel_link" />
+    <origin xyz="${chassis_length - wheel_axis_offset_x} ${-chassis_width/2} ${wheel_axis_offset_z}"
+      rpy="${pi/2} 0 0" />
+    <axis xyz="0.0 0.0 1" />
   </joint>
   <link name="FL_wheel_link">
     <visual>
       <geometry>
-        <cylinder radius="${wheel_radius}" length="${wheel_thickness}"/>
-      </geometry>
-      <origin xyz="0 0 ${wheel_thickness/2}"/>
-      <material name="black" />
-    </visual>
-    <collision>
-      <geometry>
-        <cylinder radius="${wheel_radius}" length="${wheel_thickness}"/>
-      </geometry>
-      <origin xyz="0 0 ${wheel_thickness/2}"/>
+        <cylinder radius="${wheel_radius}" length="${wheel_thickness}" />
+      </geometry>
+      <origin xyz="0 0 ${wheel_thickness/2}" />
+      <material name="black" />
+    </visual>
+    <collision>
+      <geometry>
+        <cylinder radius="${wheel_radius}" length="${wheel_thickness}" />
+      </geometry>
+      <origin xyz="0 0 ${wheel_thickness/2}" />
     </collision>
     <xacro:inertial_cylinder mass="0.020" radius="${wheel_radius}" length="${wheel_thickness}">
-      <origin xyz="0 0 ${wheel_thickness/2}"/>
+      <origin xyz="0 0 ${wheel_thickness/2}" />
     </xacro:inertial_cylinder>
   </link>
   <joint name="FR_wheel_joint" type="continuous">
-    <parent link="chassis_link"/>
-    <child link="FR_wheel_link"/>
-    <origin xyz="${chassis_length - wheel_axis_offset_x} ${chassis_width/2} ${wheel_axis_offset_z}" rpy="${pi/2} 0 0"/>
-    <axis xyz="0.0 0.0 1"/>
+    <parent link="chassis_link" />
+    <child link="FR_wheel_link" />
+    <origin xyz="${chassis_length - wheel_axis_offset_x} ${chassis_width/2} ${wheel_axis_offset_z}"
+      rpy="${pi/2} 0 0" />
+    <axis xyz="0.0 0.0 1" />
   </joint>
   <link name="FR_wheel_link">
     <visual>
       <geometry>
-        <cylinder radius="${wheel_radius}" length="${wheel_thickness}"/>
-      </geometry>
-      <origin xyz="0 0 ${-wheel_thickness/2}"/>
-      <material name="black" />
-    </visual>
-    <collision>
-      <geometry>
-        <cylinder radius="${wheel_radius}" length="${wheel_thickness}"/>
-      </geometry>
-      <origin xyz="0 0 ${-wheel_thickness/2}"/>
+        <cylinder radius="${wheel_radius}" length="${wheel_thickness}" />
+      </geometry>
+      <origin xyz="0 0 ${-wheel_thickness/2}" />
+      <material name="black" />
+    </visual>
+    <collision>
+      <geometry>
+        <cylinder radius="${wheel_radius}" length="${wheel_thickness}" />
+      </geometry>
+      <origin xyz="0 0 ${-wheel_thickness/2}" />
     </collision>
     <xacro:inertial_cylinder mass="0.020" length="${wheel_thickness}" radius="${wheel_radius}">
-      <origin xyz="0 0 ${-wheel_thickness/2}"/>
+      <origin xyz="0 0 ${-wheel_thickness/2}" />
     </xacro:inertial_cylinder>
   </link>
   <!-- LDR PLACEMENTS -->
   <joint name="center_ldr_joint" type="fixed">
-    <parent link="base_link"/>
-    <child link="center_ldr_link"/>
+    <parent link="base_link" />
+    <child link="center_ldr_link" />
   </joint>
   <link name="center_ldr_link">
     <visual>
       <geometry>
-        <box size="${ldr_height} ${ldr_height} ${ldr_height}"/>
-      </geometry>
-      <material name="red"/>
-      <origin xyz="0 0 ${-ldr_height/2}"/>
+        <box size="${ldr_height} ${ldr_height} ${ldr_height}" />
+      </geometry>
+      <material name="red" />
+      <origin xyz="0 0 ${-ldr_height/2}" />
     </visual>
   </link>
   <joint name="x1_ldr_joint" type="fixed">
-    <parent link="center_ldr_link"/>
-    <child link="x1_ldr_link"/>
-    <origin xyz="${ldr_inter_offset} 0 0"/>
+    <parent link="center_ldr_link" />
+    <child link="x1_ldr_link" />
+    <origin xyz="${ldr_inter_offset} 0 0" />
   </joint>
   <link name="x1_ldr_link">
     <visual>
       <geometry>
-        <box size="${ldr_height} ${ldr_height} ${ldr_height}"/>
-      </geometry>
-      <material name="red"/>
-      <origin xyz="0 0 ${-ldr_height/2}"/>
+        <box size="${ldr_height} ${ldr_height} ${ldr_height}" />
+      </geometry>
+      <material name="red" />
+      <origin xyz="0 0 ${-ldr_height/2}" />
     </visual>
   </link>
   <joint name="x2_ldr_joint" type="fixed">
-    <parent link="x1_ldr_link"/>
-    <child link="x2_ldr_link"/>
-    <origin xyz="${ldr_inter_offset} 0 0"/>
+    <parent link="x1_ldr_link" />
+    <child link="x2_ldr_link" />
+    <origin xyz="${ldr_inter_offset} 0 0" />
   </joint>
   <link name="x2_ldr_link">
     <visual>
       <geometry>
-        <box size="${ldr_height} ${ldr_height} ${ldr_height}"/>
-      </geometry>
-      <material name="red"/>
-      <origin xyz="0 0 ${-ldr_height/2}"/>
+        <box size="${ldr_height} ${ldr_height} ${ldr_height}" />
+      </geometry>
+      <material name="red" />
+      <origin xyz="0 0 ${-ldr_height/2}" />
     </visual>
   </link>
   <joint name="x-1_ldr_joint" type="fixed">
-    <parent link="center_ldr_link"/>
-    <child link="x-1_ldr_link"/>
-    <origin xyz="${-ldr_inter_offset} 0 0"/>
+    <parent link="center_ldr_link" />
+    <child link="x-1_ldr_link" />
+    <origin xyz="${-ldr_inter_offset} 0 0" />
   </joint>
   <link name="x-1_ldr_link">
     <visual>
       <geometry>
-        <box size="${ldr_height} ${ldr_height} ${ldr_height}"/>
-      </geometry>
-      <material name="red"/>
-      <origin xyz="0 0 ${-ldr_height/2}"/>
+        <box size="${ldr_height} ${ldr_height} ${ldr_height}" />
+      </geometry>
+      <material name="red" />
+      <origin xyz="0 0 ${-ldr_height/2}" />
     </visual>
   </link>
   <joint name="x-2_ldr_joint" type="fixed">
-    <parent link="x-1_ldr_link"/>
-    <child link="x-2_ldr_link"/>
-    <origin xyz="${-ldr_inter_offset} 0 0"/>
+    <parent link="x-1_ldr_link" />
+    <child link="x-2_ldr_link" />
+    <origin xyz="${-ldr_inter_offset} 0 0" />
   </joint>
   <link name="x-2_ldr_link">
     <visual>
       <geometry>
-        <box size="${ldr_height} ${ldr_height} ${ldr_height}"/>
-      </geometry>
-      <material name="red"/>
-      <origin xyz="0 0 ${-ldr_height/2}"/>
+        <box size="${ldr_height} ${ldr_height} ${ldr_height}" />
+      </geometry>
+      <material name="red" />
+      <origin xyz="0 0 ${-ldr_height/2}" />
     </visual>
   </link>
   <joint name="y-1_ldr_joint" type="fixed">
-    <parent link="center_ldr_link"/>
-    <child link="y-1_ldr_link"/>
-    <origin xyz="0 ${-ldr_inter_offset} 0"/>
+    <parent link="center_ldr_link" />
+    <child link="y-1_ldr_link" />
+    <origin xyz="0 ${-ldr_inter_offset} 0" />
   </joint>
   <link name="y-1_ldr_link">
     <visual>
       <geometry>
-        <box size="${ldr_height} ${ldr_height} ${ldr_height}"/>
-      </geometry>
-      <material name="red"/>
-      <origin xyz="0 0 ${-ldr_height/2}"/>
+        <box size="${ldr_height} ${ldr_height} ${ldr_height}" />
+      </geometry>
+      <material name="red" />
+      <origin xyz="0 0 ${-ldr_height/2}" />
     </visual>
   </link>
   <joint name="y-2_ldr_joint" type="fixed">
-    <parent link="y-1_ldr_link"/>
-    <child link="y-2_ldr_link"/>
-    <origin xyz="0 ${-ldr_inter_offset} 0"/>
+    <parent link="y-1_ldr_link" />
+    <child link="y-2_ldr_link" />
+    <origin xyz="0 ${-ldr_inter_offset} 0" />
   </joint>
   <link name="y-2_ldr_link">
     <visual>
       <geometry>
-        <box size="${ldr_height} ${ldr_height} ${ldr_height}"/>
-      </geometry>
-      <material name="red"/>
-      <origin xyz="0 0 ${-ldr_height/2}"/>
+        <box size="${ldr_height} ${ldr_height} ${ldr_height}" />
+      </geometry>
+      <material name="red" />
+      <origin xyz="0 0 ${-ldr_height/2}" />
     </visual>
   </link>
   <joint name="y1_ldr_joint" type="fixed">
-    <parent link="center_ldr_link"/>
-    <child link="y1_ldr_link"/>
-    <origin xyz="0 ${ldr_inter_offset} 0"/>
+    <parent link="center_ldr_link" />
+    <child link="y1_ldr_link" />
+    <origin xyz="0 ${ldr_inter_offset} 0" />
   </joint>
   <link name="y1_ldr_link">
     <visual>
       <geometry>
-        <box size="${ldr_height} ${ldr_height} ${ldr_height}"/>
-      </geometry>
-      <material name="red"/>
-      <origin xyz="0 0 ${-ldr_height/2}"/>
+        <box size="${ldr_height} ${ldr_height} ${ldr_height}" />
+      </geometry>
+      <material name="red" />
+      <origin xyz="0 0 ${-ldr_height/2}" />
     </visual>
   </link>
   <joint name="y2_ldr_joint" type="fixed">
-    <parent link="y1_ldr_link"/>
-    <child link="y2_ldr_link"/>
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
Commit message: Add mecanum drive plugin

File: ros2_ws/src/milo_sim/urdf/milo_core.urdf.xacro (robot description, xacro)
@@ -48,5 +48,5 @@
     <child link="BR_wheel_link" />
     <origin xyz="${wheel_axis_offset_x} ${chassis_width/2} ${wheel_axis_offset_z}" rpy="${pi/2} 0 0" />
-    <axis xyz="0.0 0.0 1" />
+    <axis xyz="0.0 0.0 1.0" />
   </joint>
   <link name="BR_wheel_link">
@@ -62,4 +62,13 @@
         <cylinder radius="${wheel_radius}" length="${wheel_thickness}" />
       </geometry>
+      <surface>
+      <friction>
+        <ode>
+          <mu>0.8</mu>
+          <mu2>0.5</mu2>
+          <fdir1>1 -1 0</fdir1>
+        </ode>
+      </friction>
+    </surface>
       <origin xyz="0 0 ${-wheel_thickness/2}" />
     </collision>
@@ -73,5 +82,5 @@
     <origin xyz="${wheel_axis_offset_x} ${-chassis_width/2} ${wheel_axis_offset_z}"
       rpy="${pi/2} 0 0" />
-    <axis xyz="0.0 0.0 1" />
+    <axis xyz="0.0 0.0 1.0" />
   </joint>
   <link name="BL_wheel_link">
@@ -87,4 +96,13 @@
         <cylinder radius="${wheel_radius}" length="${wheel_thickness}" />
       </geometry>
+      <surface>
+      <friction>
+        <ode>
+          <mu>0.8</mu>
+          <mu2>0.5</mu2>
+          <fdir1>-1 -1 0</fdir1>
+        </ode>
+      </friction>
+    </surface>
       <origin xyz="0 0 ${wheel_thickness/2}" />
     </collision>
@@ -98,5 +116,5 @@
     <origin xyz="${chassis_length - wheel_axis_offset_x} ${-chassis_width/2} ${wheel_axis_offset_z}"
       rpy="${pi/2} 0 0" />
-    <axis xyz="0.0 0.0 1" />
+    <axis xyz="0.0 0.0 1.0" />
   </joint>
   <link name="FL_wheel_link">
@@ -112,4 +130,13 @@
         <cylinder radius="${wheel_radius}" length="${wheel_thickness}" />
       </geometry>
+      <surface>
+      <friction>
+        <ode>
+          <mu>0.8</mu>
+          <mu2>0.5</mu2>
+          <fdir1>-1 1 0</fdir1>
+        </ode>
+      </friction>
+    </surface>
       <origin xyz="0 0 ${wheel_thickness/2}" />
     </collision>
@@ -123,5 +150,5 @@
     <origin xyz="${chassis_length - wheel_axis_offset_x} ${chassis_width/2} ${wheel_axis_offset_z}"
       rpy="${pi/2} 0 0" />
-    <axis xyz="0.0 0.0 1" />
+    <axis xyz="0.0 0.0 1.0" />
   </joint>
   <link name="FR_wheel_link">
@@ -137,4 +164,13 @@
         <cylinder radius="${wheel_radius}" length="${wheel_thickness}" />
       </geometry>
+      <surface>
+      <friction>
+        <ode>
+          <mu>0.8</mu>
+          <mu2>0.5</mu2>
+          <fdir1>1 1 0</fdir1>
+        </ode>
+      </friction>
+    </surface>
       <origin xyz="0 0 ${-wheel_thickness/2}" />
     </collision>
@@ -269,4 +305,19 @@
     </visual>
   </link>
-  <!-- GAZEBO PLUGINS -->
+  <!-- GAZEBO information -->
+  <gazebo>
+    <plugin
+      filename="gz-sim-mecanum-drive-system"
+      name="gz::sim::systems::MecanumDrive">
+      <front_left_joint>FL_wheel_joint</front_left_joint>
+      <front_right_joint>FR_wheel_joint</front_right_joint>
+      <back_left_joint>BL_wheel_joint</back_left_joint>
+      <back_right_joint>BR_wheel_joint</back_right_joint>
+      <wheel_separation>0.26</wheel_separation> <!-- Chassis width -->
+      <wheelbase>0.18</wheelbase> <!-- Chassis length - 2*wheel_offset_x -->
+      <wheel_radius>0.03</wheel_radius>
+      <min_acceleration>-5</min_acceleration>
+      <max_acceleration>5</max_acceleration>
+    </plugin>
+  </gazebo>
 </robot>
