Commit message: Add LDR sensors (as cameras)

File: ros2_ws/src/milo_sim/urdf/milo_core.urdf.xacro (robot description, xacro)
@@ -43,4 +43,11 @@
     </xacro:inertial_box>
   </link>
+  <!-- Chassis center link to link the LDRs to -->
+  <joint name="chassis_center_joint" type="fixed">
+    <parent link="chassis_link"/>
+    <child link="chassis_center_link"/>
+    <origin xyz="${chassis_length/2} 0 0" rpy="0 0 0"/>
+  </joint>
+  <link name="chassis_center_link"></link>
   <!-- WHEELS (looked at from the front of the robot) -->
   <joint name="BR_wheel_joint" type="continuous">
@@ -63,12 +70,12 @@
       </geometry>
       <surface>
-      <friction>
-        <ode>
-          <mu>0.8</mu>
-          <mu2>0.5</mu2>
-          <fdir1>1 -1 0</fdir1>
-        </ode>
-      </friction>
-    </surface>
+        <friction>
+          <ode>
+            <mu>0.8</mu>
+            <mu2>0.5</mu2>
+            <fdir1>1 -1 0</fdir1>
+          </ode>
+        </friction>
+      </surface>
       <origin xyz="0 0 ${-wheel_thickness/2}" />
     </collision>
@@ -97,12 +104,12 @@
       </geometry>
       <surface>
-      <friction>
-        <ode>
-          <mu>0.8</mu>
-          <mu2>0.5</mu2>
-          <fdir1>-1 -1 0</fdir1>
-        </ode>
-      </friction>
-    </surface>
+        <friction>
+          <ode>
+            <mu>0.8</mu>
+            <mu2>0.5</mu2>
+            <fdir1>-1 -1 0</fdir1>
+          </ode>
+        </friction>
+      </surface>
       <origin xyz="0 0 ${wheel_thickness/2}" />
     </collision>
@@ -131,12 +138,12 @@
       </geometry>
       <surface>
-      <friction>
-        <ode>
-          <mu>0.8</mu>
-          <mu2>0.5</mu2>
-          <fdir1>-1 1 0</fdir1>
-        </ode>
-      </friction>
-    </surface>
+        <friction>
+          <ode>
+            <mu>0.8</mu>
+            <mu2>0.5</mu2>
+            <fdir1>-1 1 0</fdir1>
+          </ode>
+        </friction>
+      </surface>
       <origin xyz="0 0 ${wheel_thickness/2}" />
     </collision>
@@ -165,12 +172,12 @@
       </geometry>
       <surface>
-      <friction>
-        <ode>
-          <mu>0.8</mu>
-          <mu2>0.5</mu2>
-          <fdir1>1 1 0</fdir1>
-        </ode>
-      </friction>
-    </surface>
+        <friction>
+          <ode>
+            <mu>0.8</mu>
+            <mu2>0.5</mu2>
+            <fdir1>1 1 0</fdir1>
+          </ode>
+        </friction>
+      </surface>
       <origin xyz="0 0 ${-wheel_thickness/2}" />
     </collision>
@@ -181,6 +188,7 @@
   <!-- LDR PLACEMENTS -->
   <joint name="center_ldr_joint" type="fixed">
-    <parent link="base_link" />
+    <parent link="chassis_center_link" />
     <child link="center_ldr_link" />
+    <origin xyz="0 0 ${-ldr_height/2}" rpy="0 ${pi/2} 0"/>
   </joint>
   <link name="center_ldr_link">
@@ -190,11 +198,20 @@
       </geometry>
       <material name="red" />
-      <origin xyz="0 0 ${-ldr_height/2}" />
-    </visual>
+      <origin xyz="0 0 ${-ldr_height/2}" rpy="0 0 0"/>
+    </visual>
+    <collision>
+      <geometry>
+        <box size="${ldr_height} ${ldr_height} ${ldr_height}"/>
+      </geometry>
+    </collision>
+    <xacro:inertial_box mass="0.001" x="${ldr_height}" y="${ldr_height}"
+      z="${ldr_height}">
+      <origin xyz="0 0 ${ldr_height/2}" />
+    </xacro:inertial_box>
   </link>
   <joint name="x1_ldr_joint" type="fixed">
     <parent link="center_ldr_link" />
     <child link="x1_ldr_link" />
-    <origin xyz="${ldr_inter_offset} 0 0" />
+    <origin xyz="0 0 ${ldr_inter_offset}" />
   </joint>
   <link name="x1_ldr_link">
@@ -206,9 +223,18 @@
       <origin xyz="0 0 ${-ldr_height/2}" />
     </visual>
+    <collision>
+      <geometry>
+        <box size="${ldr_height} ${ldr_height} ${ldr_height}"/>
+      </geometry>
+    </collision>
+    <xacro:inertial_box mass="0.001" x="${ldr_height}" y="${ldr_height}"
+      z="${ldr_height}">
+      <origin xyz="0 0 ${-ldr_height/2}" />
+    </xacro:inertial_box>
   </link>
   <joint name="x2_ldr_joint" type="fixed">
     <parent link="x1_ldr_link" />
     <child link="x2_ldr_link" />
-    <origin xyz="${ldr_inter_offset} 0 0" />
+    <origin xyz="0 0 ${ldr_inter_offset}" />
   </joint>
   <link name="x2_ldr_link">
@@ -220,9 +246,18 @@
       <origin xyz="0 0 ${-ldr_height/2}" />
     </visual>
+    <collision>
+      <geometry>
+        <box size="${ldr_height} ${ldr_height} ${ldr_height}"/>
+      </geometry>
+    </collision>
+    <xacro:inertial_box mass="0.001" x="${ldr_height}" y="${ldr_height}"
+      z="${ldr_height}">
+      <origin xyz="0 0 ${-ldr_height/2}" />
+    </xacro:inertial_box>
   </link>
   <joint name="x-1_ldr_joint" type="fixed">
     <parent link="center_ldr_link" />
     <child link="x-1_ldr_link" />
-    <origin xyz="${-ldr_inter_offset} 0 0" />
+    <origin xyz="0 0 ${-ldr_inter_offset}" />
   </joint>
   <link name="x-1_ldr_link">
@@ -234,9 +269,18 @@
       <origin xyz="0 0 ${-ldr_height/2}" />
     </visual>
+    <collision>
+      <geometry>
+        <box size="${ldr_height} ${ldr_height} ${ldr_height}"/>
+      </geometry>
+    </collision>
+    <xacro:inertial_box mass="0.001" x="${ldr_height}" y="${ldr_height}"
+      z="${ldr_height}">
+      <origin xyz="0 0 ${-ldr_height/2}" />
+    </xacro:inertial_box>
   </link>
   <joint name="x-2_ldr_joint" type="fixed">
     <parent link="x-1_ldr_link" />
     <child link="x-2_ldr_link" />
-    <origin xyz="${-ldr_inter_offset} 0 0" />
+    <origin xyz="0 0 ${-ldr_inter_offset}" />
   </joint>
   <link name="x-2_ldr_link">
@@ -248,4 +292,13 @@
       <origin xyz="0 0 ${-ldr_height/2}" />
     </visual>
+    <collision>
+      <geometry>
+        <box size="${ldr_height} ${ldr_height} ${ldr_height}"/>
+      </geometry>
+    </collision>
+    <xacro:inertial_box mass="0.001" x="${ldr_height}" y="${ldr_height}"
+      z="${ldr_height}">
+      <origin xyz="0 0 ${-ldr_height/2}" />
+    </xacro:inertial_box>
   </link>
   <joint name="y-1_ldr_joint" type="fixed">
@@ -262,4 +315,13 @@
       <origin xyz="0 0 ${-ldr_height/2}" />
     </visual>
+    <collision>
+      <geometry>
+        <box size="${ldr_height} ${ldr_height} ${ldr_height}"/>
+      </geometry>
+    </collision>
+    <xacro:inertial_box mass="0.001" x="${ldr_height}" y="${ldr_height}"
+      z="${ldr_height}">
+      <origin xyz="0 0 ${-ldr_height/2}" />
+    </xacro:inertial_box>
   </link>
   <joint name="y-2_ldr_joint" type="fixed">
@@ -276,4 +338,13 @@
       <origin xyz="0 0 ${-ldr_height/2}" />
     </visual>
+    <collision>
+      <geometry>
+        <box size="${ldr_height} ${ldr_height} ${ldr_height}"/>
+      </geometry>
+    </collision>
+    <xacro:inertial_box mass="0.001" x="${ldr_height}" y="${ldr_height}"
+      z="${ldr_height}">
+      <origin xyz="0 0 ${-ldr_height/2}" />
+    </xacro:inertial_box>
   </link>
   <joint name="y1_ldr_joint" type="fixed">
@@ -290,4 +361,13 @@
       <origin xyz="0 0 ${-ldr_height/2}" />
     </visual>
+    <collision>
+      <geometry>
+        <box size="${ldr_height} ${ldr_height} ${ldr_height}"/>
+      </geometry>
+    </collision>
+    <xacro:inertial_box mass="0.001" x="${ldr_height}" y="${ldr_height}"
+      z="${ldr_height}">
+      <origin xyz="0 0 ${-ldr_height/2}" />
+    </xacro:inertial_box>
   </link>
   <joint name="y2_ldr_joint" type="fixed">
@@ -304,4 +384,13 @@
       <origin xyz="0 0 ${-ldr_height/2}" />
     </visual>
+    <collision>
+      <geometry>
+        <box size="${ldr_height} ${ldr_height} ${ldr_height}"/>
+      </geometry>
+    </collision>
+    <xacro:inertial_box mass="0.001" x="${ldr_height}" y="${ldr_height}"
+      z="${ldr_height}">
+      <origin xyz="0 0 ${-ldr_height/2}" />
+    </xacro:inertial_box>
   </link>
   <!-- GAZEBO information -->
@@ -321,3 +410,131 @@
     </plugin>
   </gazebo>
+  <gazebo reference="x1_ldr_link">
+    <sensor name="front_LDR1" type="camera">
+      <camera>
+        <horizontal_fov>1.0472</horizontal_fov>
+        <image>
+          <width>10</width>
+          <height>8</height>
+        </image>
+        <clip> <!-- The range of the camera-->
+          <near>0.001</near>
+          <far>0.2</far>
+        </clip>
+      </camera>
+      <topic>milo/fldr1</topic>
+    </sensor>
+  </gazebo>
+  <gazebo reference="x2_ldr_link">
+    <sensor name="front_LDR2" type="camera">
+      <camera>
+        <horizontal_fov>1.0472</horizontal_fov>
+        <image>
+          <width>10</width>
+          <height>8</height>
+        </image>
+        <clip> <!-- The range of the camera-->
+          <near>0.001</near>
+          <far>0.2</far>
+        </clip>
+      </camera>
+      <topic>milo/fldr2</topic>
+    </sensor>
+  </gazebo>
+  <gazebo reference="x-1_ldr_link">
+    <sensor name="back_LDR1" type="camera">
+      <camera>
+        <horizontal_fov>1.0472</horizontal_fov>
+        <image>
+          <width>10</width>
+          <height>8</height>
+        </image>
+        <clip> <!-- The range of the camera-->
+          <near>0.001</near>
+          <far>0.2</far>
+        </clip>
+      </camera>
+      <topic>milo/bldr1</topic>
+    </sensor>
+  </gazebo>
+  <gazebo reference="x-2_ldr_link">
+    <sensor name="back_LDR2" type="camera">
+      <camera>
+        <horizontal_fov>1.0472</horizontal_fov>
+        <image>
+          <width>10</width>
+          <height>8</height>
+        </image>
+        <clip> <!-- The range of the camera-->
+          <near>0.001</near>
+          <far>0.2</far>
+        </clip>
+      </camera>
+      <topic>milo/bldr2</topic>
+    </sensor>
+  </gazebo>
+  <gazebo reference="y1_ldr_link">
+    <sensor name="left_LDR1" type="camera">
+      <camera>
+        <horizontal_fov>1.0472</horizontal_fov>
+        <image>
+          <width>10</width>
+          <height>8</height>
+        </image>
+        <clip> <!-- The range of the camera-->
+          <near>0.001</near>
+          <far>0.2</far>
+        </clip>
+      </camera>
+      <topic>milo/lldr1</topic>
+    </sensor>
+  </gazebo>
+  <gazebo reference="y-1_ldr_link">
+    <sensor name="right_LDR1" type="camera">
+      <camera>
+        <horizontal_fov>1.0472</horizontal_fov>
+        <image>
+          <width>10</width>
+          <height>8</height>
+        </image>
+        <clip> <!-- The range of the camera-->
+          <near>0.001</near>
+          <far>0.2</far>
+        </clip>
+      </camera>
+      <topic>milo/rldr1</topic>
+    </sensor>
+  </gazebo>
+  <gazebo reference="y2_ldr_link">
+    <sensor name="left_LDR2" type="camera">
+      <camera>
+        <horizontal_fov>1.0472</horizontal_fov>
+        <image>
+          <width>10</width>
+          <height>8</height>
+        </image>
+        <clip> <!-- The range of the camera-->
+          <near>0.001</near>
+          <far>0.2</far>
+        </clip>
+      </camera>
+      <topic>milo/lldr2</topic>
+    </sensor>
+  </gazebo>
+  <gazebo reference="y-2_ldr_link">
+    <sensor name="right_LDR2" type="camera">
+      <camera>
+        <horizontal_fov>1.0472</horizontal_fov>
+        <image>
+          <width>10</width>
+          <height>8</height>
+        </image>
+        <clip> <!-- The range of the camera-->
+          <near>0.001</near>
+          <far>0.2</far>
+        </clip>
+      </camera>
+      <topic>milo/rldr2</topic>
+    </sensor>
+  </gazebo>
 </robot>

Commit message: Update urdf and launch file

File: ros2_ws/src/milo_sim/urdf/milo_core.urdf.xacro (robot description, xacro)
@@ -13,6 +13,6 @@
   <xacro:property name="wheel_radius" value="0.03" />
   <xacro:property name="wheel_thickness" value="0.025" />
-  <xacro:property name="ldr_inter_offset" value="0.02" />
-  <xacro:property name="ldr_height" value="0.01" />
+  <xacro:property name="ldr_inter_offset" value="0.025" />
+  <xacro:property name="ldr_height" value="0.005" />
   <!-- World link without inertia required by rviz -->
   <link name="base_link">
@@ -411,7 +411,7 @@
   </gazebo>
   <gazebo reference="x1_ldr_link">
-    <sensor name="front_LDR1" type="camera">
-      <camera>
-        <horizontal_fov>1.0472</horizontal_fov>
+    <sensor name="f1" type="camera">
+      <camera>
+        <horizontal_fov>2.09439510239</horizontal_fov>
         <image>
           <width>10</width>
@@ -428,7 +428,7 @@
   </gazebo>
   <gazebo reference="x2_ldr_link">
-    <sensor name="front_LDR2" type="camera">
-      <camera>
-        <horizontal_fov>1.0472</horizontal_fov>
+    <sensor name="f0" type="camera">
+      <camera>
+        <horizontal_fov>2.09439510239</horizontal_fov>
         <image>
           <width>10</width>
@@ -445,7 +445,7 @@
   </gazebo>
   <gazebo reference="x-1_ldr_link">
-    <sensor name="back_LDR1" type="camera">
-      <camera>
-        <horizontal_fov>1.0472</horizontal_fov>
+    <sensor name="f2" type="camera">
+      <camera>
+        <horizontal_fov>2.09439510239</horizontal_fov>
         <image>
           <width>10</width>
@@ -462,7 +462,7 @@
   </gazebo>
   <gazebo reference="x-2_ldr_link">
-    <sensor name="back_LDR2" type="camera">
-      <camera>
-        <horizontal_fov>1.0472</horizontal_fov>
+    <sensor name="f3" type="camera">
+      <camera>
+        <horizontal_fov>2.09439510239</horizontal_fov>
         <image>
           <width>10</width>
@@ -479,7 +479,7 @@
   </gazebo>
   <gazebo reference="y1_ldr_link">
-    <sensor name="left_LDR1" type="camera">
-      <camera>
-        <horizontal_fov>1.0472</horizontal_fov>
+    <sensor name="l1" type="camera">
+      <camera>
+        <horizontal_fov>2.09439510239</horizontal_fov>
         <image>
           <width>10</width>
@@ -496,7 +496,7 @@
   </gazebo>
   <gazebo reference="y-1_ldr_link">
-    <sensor name="right_LDR1" type="camera">
-      <camera>
-        <horizontal_fov>1.0472</horizontal_fov>
+    <sensor name="l2" type="camera">
+      <camera>
+        <horizontal_fov>2.09439510239</horizontal_fov>
         <image>
           <width>10</width>
@@ -513,7 +513,7 @@
   </gazebo>
   <gazebo reference="y2_ldr_link">
-    <sensor name="left_LDR2" type="camera">
-      <camera>
-        <horizontal_fov>1.0472</horizontal_fov>
+    <sensor name="l0" type="camera">
+      <camera>
+        <horizontal_fov>2.09439510239</horizontal_fov>
         <image>
           <width>10</width>
@@ -530,7 +530,7 @@
   </gazebo>
   <gazebo reference="y-2_ldr_link">
-    <sensor name="right_LDR2" type="camera">
-      <camera>
-        <horizontal_fov>1.0472</horizontal_fov>
+    <sensor name="l3" type="camera">
+      <camera>
+        <horizontal_fov>2.09439510239</horizontal_fov>
         <image>
           <width>10</width>

Commit message: Fix not being able to move laterally

File: ros2_ws/src/milo_sim/urdf/milo_core.urdf.xacro (robot description, xacro)
@@ -1,4 +1,4 @@
 <?xml version="1.0"?>
-<robot xmlns:xacro="http://www.ros.org/wiki/xacro">
+<robot xmlns:xacro="http://www.ros.org/wiki/xacro" xmlns:gz="http://gazebosim.org/schema">
   <!-- Include useful macros -->
   <xacro:include filename="inertial_macros.xacro" />
@@ -54,6 +54,8 @@
     <parent link="chassis_link" />
     <child link="BR_wheel_link" />
-    <origin xyz="${wheel_axis_offset_x} ${chassis_width/2} ${wheel_axis_offset_z}" rpy="${pi/2} 0 0" />
-    <axis xyz="0.0 0.0 1.0" />
+    <origin xyz="${wheel_axis_offset_x} ${chassis_width/2 + wheel_thickness} ${wheel_axis_offset_z}" rpy="${-pi/2} 0 0" />
+    <axis xyz="0.0 0.0 -1.0" />
+    <limit effort="10000" velocity="10"/>
+    <dynamics damping="1.0" friction="1.0"/>
   </joint>
   <link name="BR_wheel_link">
@@ -69,13 +71,4 @@
         <cylinder radius="${wheel_radius}" length="${wheel_thickness}" />
       </geometry>
-      <surface>
-        <friction>
-          <ode>
-            <mu>0.8</mu>
-            <mu2>0.5</mu2>
-            <fdir1>1 -1 0</fdir1>
-          </ode>
-        </friction>
-      </surface>
       <origin xyz="0 0 ${-wheel_thickness/2}" />
     </collision>
@@ -90,4 +83,6 @@
       rpy="${pi/2} 0 0" />
     <axis xyz="0.0 0.0 1.0" />
+    <limit effort="10000" velocity="10"/>
+    <dynamics damping="1.0" friction="1.0"/>
   </joint>
   <link name="BL_wheel_link">
@@ -103,13 +98,4 @@
         <cylinder radius="${wheel_radius}" length="${wheel_thickness}" />
       </geometry>
-      <surface>
-        <friction>
-          <ode>
-            <mu>0.8</mu>
-            <mu2>0.5</mu2>
-            <fdir1>-1 -1 0</fdir1>
-          </ode>
-        </friction>
-      </surface>
       <origin xyz="0 0 ${wheel_thickness/2}" />
     </collision>
@@ -124,4 +110,6 @@
       rpy="${pi/2} 0 0" />
     <axis xyz="0.0 0.0 1.0" />
+    <limit effort="10000" velocity="10"/>
+    <dynamics damping="1.0" friction="1.0"/>
   </joint>
   <link name="FL_wheel_link">
@@ -137,13 +125,4 @@
         <cylinder radius="${wheel_radius}" length="${wheel_thickness}" />
       </geometry>
-      <surface>
-        <friction>
-          <ode>
-            <mu>0.8</mu>
-            <mu2>0.5</mu2>
-            <fdir1>-1 1 0</fdir1>
-          </ode>
-        </friction>
-      </surface>
       <origin xyz="0 0 ${wheel_thickness/2}" />
     </collision>
@@ -155,7 +134,9 @@
     <parent link="chassis_link" />
     <child link="FR_wheel_link" />
-    <origin xyz="${chassis_length - wheel_axis_offset_x} ${chassis_width/2} ${wheel_axis_offset_z}"
-      rpy="${pi/2} 0 0" />
-    <axis xyz="0.0 0.0 1.0" />
+    <origin xyz="${chassis_length - wheel_axis_offset_x} ${chassis_width/2 + wheel_thickness} ${wheel_axis_offset_z}"
+      rpy="${-pi/2} 0 0" />
+    <axis xyz="0.0 0.0 -1.0" />
+    <limit effort="10000" velocity="10"/>
+    <dynamics damping="1.0" friction="1.0"/>
   </joint>
   <link name="FR_wheel_link">
@@ -171,13 +152,4 @@
         <cylinder radius="${wheel_radius}" length="${wheel_thickness}" />
       </geometry>
-      <surface>
-        <friction>
-          <ode>
-            <mu>0.8</mu>
-            <mu2>0.5</mu2>
-            <fdir1>1 1 0</fdir1>
-          </ode>
-        </friction>
-      </surface>
       <origin xyz="0 0 ${-wheel_thickness/2}" />
     </collision>
@@ -425,5 +397,5 @@
           <type>gaussian</type>
           <mean>0.0</mean>
-          <stddev>0.35</stddev>
+          <stddev>0.2</stddev>
         </noise>
       </camera>
@@ -447,5 +419,5 @@
           <type>gaussian</type>
           <mean>0.0</mean>
-          <stddev>0.35</stddev>
+          <stddev>0.2</stddev>
         </noise>
       </camera>
@@ -469,5 +441,5 @@
           <type>gaussian</type>
           <mean>0.0</mean>
-          <stddev>0.35</stddev>
+          <stddev>0.2</stddev>
         </noise>
       </camera>
@@ -491,5 +463,5 @@
           <type>gaussian</type>
           <mean>0.0</mean>
-          <stddev>0.35</stddev>
+          <stddev>0.2</stddev>
         </noise>
       </camera>
@@ -513,5 +485,5 @@
           <type>gaussian</type>
           <mean>0.0</mean>
-          <stddev>0.35</stddev>
+          <stddev>0.2</stddev>
         </noise>
       </camera>
@@ -535,5 +507,5 @@
           <type>gaussian</type>
           <mean>0.0</mean>
-          <stddev>0.35</stddev>
+          <stddev>0.2</stddev>
         </noise>
       </camera>
@@ -557,5 +529,5 @@
           <type>gaussian</type>
           <mean>0.0</mean>
-          <stddev>0.35</stddev>
+          <stddev>0.2</stddev>
         </noise>
       </camera>
@@ -579,5 +551,5 @@
           <type>gaussian</type>
           <mean>0.0</mean>
-          <stddev>0.35</stddev>
+          <stddev>0.2</stddev>
         </noise>
       </camera>
@@ -586,3 +558,61 @@
     </sensor>
   </gazebo>
+  <!-- STEP 6 - Gazebo frictions and colors -->
+  <gazebo reference='FL_wheel_link'>
+    <collision>
+      <surface>
+        <friction>
+          <ode>
+            <mu>1.5</mu>
+            <mu2>0.0</mu2>
+            <fdir1 gz:expressed_in="base_link">1 -1 0</fdir1>
+          </ode>
+        </friction>
+      </surface>
+    </collision>
+  </gazebo>
+  <gazebo reference='BL_wheel_link'>
+    <collision>
+      <surface>
+        <friction>
+          <ode>
+            <mu>1.5</mu>
+            <mu2>0.0</mu2>
+            <fdir1 gz:expressed_in="base_link">1 1 0</fdir1>
+          </ode>
+        </friction>
+      </surface>
+    </collision>
+  </gazebo>
+  <gazebo reference='FR_wheel_link'>
+    <collision>
+      <surface>
+        <friction>
+          <ode>
+            <mu>1.5</mu>
+            <mu2>0.0</mu2>
+            <fdir1 gz:expressed_in="base_link">1 1 0</fdir1>
+          </ode>
+        </friction>
+      </surface>
+    </collision>
+  </gazebo>
+  <gazebo reference='BR_wheel_link'>
+    <collision>
+      <surface>
+        <friction>
+          <ode>
+            <mu>1.5</mu>
+            <mu2>0.0</mu2>
+            <fdir1 gz:expressed_in="base_link">1 -1 0</fdir1>
+          </ode>
+        </friction>
+      </surface>
+    </collision>
+  </gazebo>
+  <gazebo reference="chassis_link">
+    <mu1>0.000002</mu1>
+    <mu2>0.000002</mu2>
+    <!-- <material>Gazebo/Red</material> -->
+  </gazebo>
 </robot>
