Commit message: /

File: ros2_ws/src/milo_sim/urdf/milo_circular.urdf.xacro (robot description, xacro)
@@ -160,9 +160,9 @@
   </link>
   <!-- LDR PLACEMENTS -->
-  <xacro:macro name="ldr_joint_and_link" params="name angle">
+  <xacro:macro name="ldr_joint_and_link" params="name angle radius">
     <joint name="${name}_joint" type="fixed">
       <parent link="chassis_center_link"/>
       <child link="${name}_link"/>
-      <origin xyz="${ldr_radius * cos(angle)} ${ldr_radius * sin(angle)} 0" rpy="0 ${pi/2} 0"/>
+      <origin xyz="${radius * cos(angle)} ${radius * sin(angle)} 0" rpy="0 ${pi/2} 0"/>
     </joint>
     <link name="${name}_link">
@@ -184,12 +184,14 @@
     </link>
   </xacro:macro>
-  <xacro:ldr_joint_and_link name="ldr1" angle="0"/>
-  <xacro:ldr_joint_and_link name="ldr2" angle="${pi/4}"/>
-  <xacro:ldr_joint_and_link name="ldr3" angle="${pi/2}"/>
-  <xacro:ldr_joint_and_link name="ldr4" angle="${3*pi/4}"/>
-  <xacro:ldr_joint_and_link name="ldr5" angle="${pi}"/>
-  <xacro:ldr_joint_and_link name="ldr6" angle="${5*pi/4}"/>
-  <xacro:ldr_joint_and_link name="ldr7" angle="${3*pi/2}"/>
-  <xacro:ldr_joint_and_link name="ldr8" angle="${7*pi/4}"/>
+  <xacro:ldr_joint_and_link name="ldr1" angle="0" radius="${ldr_radius}"/>
+  <xacro:ldr_joint_and_link name="ldr2" angle="${pi/4}" radius="${ldr_radius}"/>
+  <xacro:ldr_joint_and_link name="ldr3" angle="${pi/2}" radius="${ldr_radius}"/>
+  <xacro:ldr_joint_and_link name="ldr4" angle="${3*pi/4}" radius="${ldr_radius}"/>
+  <xacro:ldr_joint_and_link name="ldr5" angle="${pi}" radius="${ldr_radius}"/>
+  <xacro:ldr_joint_and_link name="ldr6" angle="${5*pi/4}" radius="${ldr_radius}"/>
+  <xacro:ldr_joint_and_link name="ldr7" angle="${3*pi/2}" radius="${ldr_radius}"/>
+  <xacro:ldr_joint_and_link name="ldr8" angle="${7*pi/4}" radius="${ldr_radius}"/>
+  <xacro:ldr_joint_and_link name="ldr9" angle="${pi/4}" radius="0.10"/>
+  <xacro:ldr_joint_and_link name="ldr10" angle="${5*pi/4}" radius="0.10"/>
   <!-- GAZEBO information -->
   <gazebo>
@@ -204,6 +206,6 @@
       <wheelbase>0.18</wheelbase> <!-- Chassis length - 2*wheel_offset_x -->
       <wheel_radius>0.03</wheel_radius>
-      <min_acceleration>-5</min_acceleration>
-      <max_acceleration>5</max_acceleration>
+      <min_acceleration>-10</min_acceleration>
+      <max_acceleration>10</max_acceleration>
     </plugin>
   </gazebo>
@@ -381,4 +383,48 @@
       </camera>
       <topic>milo/ldr8</topic>
+      <update_rate>7</update_rate>
+    </sensor>
+  </gazebo>
+  <gazebo reference="ldr9_link">
+    <sensor name="8" type="camera">
+      <camera>
+        <horizontal_fov>1.25</horizontal_fov>
+        <image>
+          <width>10</width>
+          <height>8</height>
+        </image>
+        <clip> <!-- The range of the camera-->
+          <near>0.001</near>
+          <far>0.2</far>
+        </clip>
+        <noise>
+          <type>gaussian</type>
+          <mean>0.0</mean>
+          <stddev>0.2</stddev>
+        </noise>
+      </camera>
+      <topic>milo/ldr9</topic>
+      <update_rate>7</update_rate>
+    </sensor>
+  </gazebo>
+  <gazebo reference="ldr10_link">
+    <sensor name="9" type="camera">
+      <camera>
+        <horizontal_fov>1.25</horizontal_fov>
+        <image>
+          <width>10</width>
+          <height>8</height>
+        </image>
+        <clip> <!-- The range of the camera-->
+          <near>0.001</near>
+          <far>0.2</far>
+        </clip>
+        <noise>
+          <type>gaussian</type>
+          <mean>0.0</mean>
+          <stddev>0.2</stddev>
+        </noise>
+      </camera>
+      <topic>milo/ldr10</topic>
       <update_rate>7</update_rate>
     </sensor>

Commit message: Working circular ldr algorithm

File: ros2_ws/src/milo_sim/urdf/milo_circular.urdf.xacro (robot description, xacro)
@@ -13,5 +13,4 @@
   <xacro:property name="wheel_radius" value="0.03" />
   <xacro:property name="wheel_thickness" value="0.025" />
-  <xacro:property name="ldr_inter_offset" value="0.025" />
   <xacro:property name="ldr_height" value="0.005" />
   <xacro:property name="ldr_radius" value="0.035"/>
@@ -58,5 +57,4 @@
     <axis xyz="0.0 0.0 -1.0" />
     <limit effort="10000" velocity="10"/>
-    <dynamics damping="1.0" friction="1.0"/>
   </joint>
   <link name="BR_wheel_link">
@@ -85,5 +83,4 @@
     <axis xyz="0.0 0.0 1.0" />
     <limit effort="10000" velocity="10"/>
-    <dynamics damping="1.0" friction="1.0"/>
   </joint>
   <link name="BL_wheel_link">
@@ -112,5 +109,4 @@
     <axis xyz="0.0 0.0 1.0" />
     <limit effort="10000" velocity="10"/>
-    <dynamics damping="1.0" friction="1.0"/>
   </joint>
   <link name="FL_wheel_link">
@@ -139,5 +135,4 @@
     <axis xyz="0.0 0.0 -1.0" />
     <limit effort="10000" velocity="10"/>
-    <dynamics damping="1.0" friction="1.0"/>
   </joint>
   <link name="FR_wheel_link">
@@ -184,14 +179,14 @@
     </link>
   </xacro:macro>
-  <xacro:ldr_joint_and_link name="ldr1" angle="0" radius="${ldr_radius}"/>
-  <xacro:ldr_joint_and_link name="ldr2" angle="${pi/4}" radius="${ldr_radius}"/>
-  <xacro:ldr_joint_and_link name="ldr3" angle="${pi/2}" radius="${ldr_radius}"/>
-  <xacro:ldr_joint_and_link name="ldr4" angle="${3*pi/4}" radius="${ldr_radius}"/>
-  <xacro:ldr_joint_and_link name="ldr5" angle="${pi}" radius="${ldr_radius}"/>
-  <xacro:ldr_joint_and_link name="ldr6" angle="${5*pi/4}" radius="${ldr_radius}"/>
-  <xacro:ldr_joint_and_link name="ldr7" angle="${3*pi/2}" radius="${ldr_radius}"/>
-  <xacro:ldr_joint_and_link name="ldr8" angle="${7*pi/4}" radius="${ldr_radius}"/>
-  <xacro:ldr_joint_and_link name="ldr9" angle="${pi/4}" radius="0.10"/>
-  <xacro:ldr_joint_and_link name="ldr10" angle="${5*pi/4}" radius="0.10"/>
+  <xacro:ldr_joint_and_link name="ldr1" angle="${pi}" radius="${ldr_radius}"/>
+  <xacro:ldr_joint_and_link name="ldr2" angle="${5*pi/4}" radius="${ldr_radius}"/>
+  <xacro:ldr_joint_and_link name="ldr3" angle="${3*pi/2}" radius="${ldr_radius}"/>
+  <xacro:ldr_joint_and_link name="ldr4" angle="${7*pi/4}" radius="${ldr_radius}"/>
+  <xacro:ldr_joint_and_link name="ldr5" angle="0" radius="${ldr_radius}"/>
+  <xacro:ldr_joint_and_link name="ldr6" angle="${pi/4}" radius="${ldr_radius}"/>
+  <xacro:ldr_joint_and_link name="ldr7" angle="${pi/2}" radius="${ldr_radius}"/>
+  <xacro:ldr_joint_and_link name="ldr8" angle="${3*pi/4}" radius="${ldr_radius}"/>
+  <!-- <xacro:ldr_joint_and_link name="ldr9" angle="${5*pi/4}" radius="0.16"/>
+  <xacro:ldr_joint_and_link name="ldr10" angle="${pi/4}" radius="0.16"/> -->
   <!-- GAZEBO information -->
   <gazebo>
@@ -215,6 +210,6 @@
         <horizontal_fov>1.25</horizontal_fov>
         <image>
-          <width>10</width>
-          <height>8</height>
+          <width>6</width>
+          <height>6</height>
         </image>
         <clip> <!-- The range of the camera-->
@@ -229,5 +224,5 @@
       </camera>
       <topic>milo/ldr1</topic>
-      <update_rate>7</update_rate>
+      <update_rate>30</update_rate>
     </sensor>
   </gazebo>
@@ -237,6 +232,6 @@
         <horizontal_fov>1.25</horizontal_fov>
         <image>
-          <width>10</width>
-          <height>8</height>
+          <width>6</width>
+          <height>6</height>
         </image>
         <clip> <!-- The range of the camera-->
@@ -251,5 +246,5 @@
       </camera>
       <topic>milo/ldr2</topic>
-      <update_rate>7</update_rate>
+      <update_rate>30</update_rate>
     </sensor>
   </gazebo>
@@ -259,6 +254,6 @@
         <horizontal_fov>1.25</horizontal_fov>
         <image>
-          <width>10</width>
-          <height>8</height>
+          <width>6</width>
+          <height>6</height>
         </image>
         <clip> <!-- The range of the camera-->
@@ -273,5 +268,5 @@
       </camera>
       <topic>milo/ldr3</topic>
-      <update_rate>7</update_rate>
+      <update_rate>30</update_rate>
     </sensor>
   </gazebo>
@@ -281,6 +276,6 @@
         <horizontal_fov>1.25</horizontal_fov>
         <image>
-          <width>10</width>
-          <height>8</height>
+          <width>6</width>
+          <height>6</height>
         </image>
         <clip> <!-- The range of the camera-->
@@ -295,5 +290,5 @@
       </camera>
       <topic>milo/ldr4</topic>
-      <update_rate>7</update_rate>
+      <update_rate>30</update_rate>
     </sensor>
   </gazebo>
@@ -303,6 +298,6 @@
         <horizontal_fov>1.25</horizontal_fov>
         <image>
-          <width>10</width>
-          <height>8</height>
+          <width>6</width>
+          <height>6</height>
         </image>
         <clip> <!-- The range of the camera-->
@@ -317,5 +312,5 @@
       </camera>
       <topic>milo/ldr5</topic>
-      <update_rate>7</update_rate>
+      <update_rate>30</update_rate>
     </sensor>
   </gazebo>
@@ -325,6 +320,6 @@
         <horizontal_fov>1.25</horizontal_fov>
         <image>
-          <width>10</width>
-          <height>8</height>
+          <width>6</width>
+          <height>6</height>
         </image>
         <clip> <!-- The range of the camera-->
@@ -339,5 +334,5 @@
       </camera>
       <topic>milo/ldr6</topic>
-      <update_rate>7</update_rate>
+      <update_rate>30</update_rate>
     </sensor>
   </gazebo>
@@ -347,6 +342,6 @@
         <horizontal_fov>1.25</horizontal_fov>
         <image>
-          <width>10</width>
-          <height>8</height>
+          <width>6</width>
+          <height>6</height>
         </image>
         <clip> <!-- The range of the camera-->
@@ -361,5 +356,5 @@
       </camera>
       <topic>milo/ldr7</topic>
-      <update_rate>7</update_rate>
+      <update_rate>30</update_rate>
     </sensor>
   </gazebo>
@@ -369,6 +364,6 @@
         <horizontal_fov>1.25</horizontal_fov>
         <image>
-          <width>10</width>
-          <height>8</height>
+          <width>6</width>
+          <height>6</height>
         </image>
         <clip> <!-- The range of the camera-->
@@ -383,16 +378,16 @@
       </camera>
       <topic>milo/ldr8</topic>
-      <update_rate>7</update_rate>
-    </sensor>
-  </gazebo>
-  <gazebo reference="ldr9_link">
+      <update_rate>30</update_rate>
+    </sensor>
+  </gazebo>
+  <!-- <gazebo reference="ldr9_link">
     <sensor name="8" type="camera">
       <camera>
         <horizontal_fov>1.25</horizontal_fov>
         <image>
-          <width>10</width>
-          <height>8</height>
-        </image>
-        <clip> <!-- The range of the camera-->
+          <width>6</width>
+          <height>6</height>
+        </image>
+        <clip>
           <near>0.001</near>
           <far>0.2</far>
@@ -405,5 +400,5 @@
       </camera>
       <topic>milo/ldr9</topic>
-      <update_rate>7</update_rate>
+      <update_rate>30</update_rate>
     </sensor>
   </gazebo>
@@ -413,8 +408,8 @@
         <horizontal_fov>1.25</horizontal_fov>
         <image>
-          <width>10</width>
-          <height>8</height>
-        </image>
-        <clip> <!-- The range of the camera-->
+          <width>6</width>
+          <height>6</height>
+        </image>
+        <clip>
           <near>0.001</near>
           <far>0.2</far>
@@ -427,7 +422,7 @@
       </camera>
       <topic>milo/ldr10</topic>
-      <update_rate>7</update_rate>
-    </sensor>
-  </gazebo>
+      <update_rate>30</update_rate>
+    </sensor>
+  </gazebo> -->
   <!-- STEP 6 - Gazebo frictions and colors -->
   <gazebo reference='FL_wheel_link'>
